File: hardware/intercom.kicad_pcb (KiCad board)
At the start: 2 copper layers, 101.3 x 39.9 mm, 42 parts, among them J1 Conn_02x02_Odd_Even, SW1 SW_Push, SW2 POWER, U1 MAX98357A, U2 TPS61088

Commit message: further refine pcb
Parts:
- moved SW1 1.25 mm to (106.8, 103.2)
- moved C24 1.00 mm to (80.5, 86.0)
- moved C22 1.00 mm to (85.0, 86.0)
- moved C8 1.00 mm to (94.0, 86.0)
- moved R20 1.00 mm to (89.5, 86.0)
Connections:
- MK1 pad 1: Net-(MK1-WS) -> Net-(A1-D2)
- MK1 pad 2: Net-(A1-D3) -> GND
- MK1 pad 4: Net-(A1-D2) -> Net-(A1-D3)
- MK1 pad 6: unconnected-(MK1-SD-Pad6) -> Net-(A1-D4)
- R2 pad 2: Net-(A1-D2) -> Net-(A1-D3)
- R3 pad 1: Net-(A1-D4) -> Net-(A1-D2)
- R3 pad 2: Net-(MK1-WS) -> Net-(A1-D2)
Routing:
- net Net-(A1-D3): track 18.5 -> 38.3 mm, vias 0 -> 2
- net Net-(A1-D4): track 8.49 -> 19.0 mm, vias 0 -> 1
- net Net-(A1-D2): track 31.8 -> 23.0 mm, vias 3 -> 2
- net Net-(MK1-WS): track 7.13 -> 0.00 mm, vias 1 -> 0
- net GND: track 0.00 -> 4.37 mm
- net +5V: track 113.6 -> 117.1 mm
- net Net-(C22-Pad2): track 40.3 -> 38.2 mm
- net Net-(A1-D7): track 54.9 -> 56.2 mm
- net Net-(U2-BOOT): track 5.36 -> 4.36 mm
- net Net-(U2-FSW): track 5.33 -> 4.62 mm
- net Net-(A1-D8): track 47.6 -> 47.1 mm
Other:
- board text added: "ARBITER INTERCOM"
- board text added: "AUG 2026"
- board text added: "DESIGNED BY TYLER RECKART"
- board text added: "MICROPHONE"
- board text added: "MODEL 1.14"
- board text added: "SPKR VOLUME"
- board text added: "USB/DATA"
- board text removed: "ARBITER MODEL 114"
- board text removed: "DATA"
- board text removed: "INPUT"
- board text removed: "USB"
