File: hardware/intercom.kicad_pcb (KiCad board)
At the start: 2 copper layers, 101.3 x 39.9 mm, 42 parts, among them J1 Conn_02x02_Odd_Even, SW1 SW_Push, SW2 POWER, U1 MAX98357A, U2 TPS61088

Commit message: improve speech patterns
Parts:
- FB1, FB2: value FerriteBead -> 600Ω@100MHz
- R22: value 178k -> 180k
