File: hardware/intercom.kicad_sch (KiCad schematic)
At the start: 19 parts, among them J1 Conn_02x02_Odd_Even, SW1 SW_Push_45deg, U1 MAX98357A

Commit message: design rev-a pcb
Parts:
- added H1, H2, H3, H4: MountingHole_Pad, MountingHole:MountingHole_2.2mm_M2_Pad, symbol Mechanical:MountingHole_Pad
- C2, C3, C5, C6, C7, C8: footprint (none) -> Capacitor_SMD:C_0805_2012Metric_Pad1.18x1.45mm_HandSolder
- D1: value LED -> LED red; footprint (none) -> LED_THT:LED_D5.0mm
- FB1, FB2: footprint (none) -> Inductor_SMD:L_0805_2012Metric_Pad1.05x1.20mm_HandSolder
- J1: value Conn_02x02_Odd_Even -> Conn_01x02; footprint (none) -> Connector_JST:JST_PH_S2B-PH-K_1x02_P2.00mm_Horizontal; symbol Connector_Generic:Conn_02x02_Odd_Even -> Connector_Generic:Conn_01x02
- R1, R2, R3, R4: footprint (none) -> Resistor_SMD:R_0805_2012Metric_Pad1.20x1.40mm_HandSolder
- RV1: footprint (none) -> Potentiometer_THT:Potentiometer_Bourns_PTV09A-1_Single_Vertical
- SW1: footprint (none) -> Button_Switch_THT:SW_PUSH_6mm
- U1: footprint Package_DFN_QFN:TQFN-16-1EP_3x3mm_P0.5mm_EP1.23x1.23mm -> Package_DFN_QFN:TQFN-16-1EP_3x3mm_P0.5mm_EP1.23x1.23mm_ThermalVias
Connections:
- net at C6.2, FB2.2: now also J1.2 (Pin_2); no longer J1.3 (Pin_3)
- no-connect marks 18 -> 16

Commit message: further refine pcb
Connections:
- net GND: now also MK1.2 (LR), U1.17 (PAD)
- net at MK1.4 (SCK), R2.2: now also A1.6 (D3); no longer A1.5 (D2)
- net at R3.1: now also A1.5 (D2), MK1.1 (WS), R3.2; no longer A1.7 (D4)
- net at MK1.6 (SD): now also A1.7 (D4)
- net Net-(J1-Pin_3): now reaches C6.2, FB2.2, J1.2 (Pin_2)
- no-connect marks 16 -> 21
Other:
- moved on the sheet: H4
