File: hardware/rev-b/intercom.kicad_sch (KiCad schematic)
At the start: 23 parts, among them J1 Conn_01x02, SW1 SW_Push_45deg, U1 MAX98357A

Commit message: improve speech patterns
Parts:
- removed A1: Arduino_Nano_ESP32, Module:Arduino_Nano, symbol MCU_Module:Arduino_Nano_ESP32
- removed SW1: SW_Push_45deg, Button_Switch_THT:SW_PUSH_6mm, symbol Switch:SW_Push_45deg
- added J4: PTT, Connector_JST:JST_SH_SM02B-SRSS-TB_1x02-1MP_P1.00mm_Horizontal, symbol Connector_Generic:Conn_01x02
- RV1: footprint Potentiometer_THT:Potentiometer_Bourns_PTV09A-1_Single_Vertical -> Potentiometer_THT:Potentiometer_Piher_PT-10-H01_Horizontal; now fitted
Connections:
- net GND: now also J4.2 (Pin_2)
- net THINK_LED: now reaches R1.1
- net SPK_DIN: now reaches U1.1 (DIN)
- net AMP_SD: now reaches R4.2
- net +3.3V: now reaches C2.2, C3.2, RV1.1
- net VOLUME: now reaches RV1.2
- net MIC_WS: now reaches MK1.1 (WS), R3.1, R3.2
- net MIC_BCLK: now reaches MK1.4 (SCK), R2.2
- net MIC_SD: now reaches MK1.6 (SD)
- net SPK_WS: now reaches U1.14 (LRCLK)
- net SPK_BCLK: now reaches U1.16 (BCLK)
- new net PTT: J4.1 (Pin_1)
- no-connect marks 21 -> 5
Other:
- added sheet MCU (mcu.kicad_sch)
- added sheet USB power (usb_power.kicad_sch)

Commit message: update rev-b
Parts:
- removed H1, H2, H3, H4: MountingHole_Pad, MountingHole:MountingHole_2.2mm_M2_Pad, symbol Mechanical:MountingHole_Pad
- removed R4: 1M, Resistor_SMD:R_0805_2012Metric_Pad1.20x1.40mm_HandSolder, symbol Device:R_US
- C2: footprint Capacitor_SMD:C_0805_2012Metric_Pad1.18x1.45mm_HandSolder -> Capacitor_SMD:C_0402_1005Metric
- C3, C5, C6, C7: footprint Capacitor_SMD:C_0805_2012Metric_Pad1.18x1.45mm_HandSolder -> Capacitor_SMD:C_0201_0603Metric
- C8: footprint Capacitor_SMD:C_0805_2012Metric_Pad1.18x1.45mm_HandSolder -> Capacitor_SMD:C_0603_1608Metric
- D1: footprint LED_THT:LED_D5.0mm -> LED_SMD:LED_0402_1005Metric; now fitted
- J1: footprint Connector_JST:JST_PH_S2B-PH-K_1x02_P2.00mm_Horizontal -> Connector_JST:JST_PH_S2B-PH-SM4-TB_1x02-1MP_P2.00mm_Horizontal; now fitted
- J4: value PTT -> PTT BREAKOUT; footprint Connector_JST:JST_SH_SM02B-SRSS-TB_1x02-1MP_P1.00mm_Horizontal -> Connector_JST:JST_PH_S2B-PH-SM4-TB_1x02-1MP_P2.00mm_Horizontal
- J5: renamed from RV1; value A50K -> VOLUME BREAKOUT; footprint Potentiometer_THT:Potentiometer_Piher_PT-10-H01_Horizontal -> Connector_JST:JST_PH_S3B-PH-SM4-TB_1x03-1MP_P2.00mm_Horizontal; symbol Device:R_Potentiometer_US -> Connector_Generic:Conn_01x03
- R1, R2, R3: footprint Resistor_SMD:R_0805_2012Metric_Pad1.20x1.40mm_HandSolder -> Resistor_SMD:R_0201_0603Metric
- U1: value MAX98357A -> MAX98357AETE+T
Connections:
- net +3.3V: now also C2.1, C3.1, J5.3 (Pin_3), MK1.5 (VDD); no longer C2.2, C3.2, J5.1
- net AMP_SD: now also U1.4 (~{SD_MODE})
- net GND: now also C2.2, C3.2, J5.1 (Pin_1); no longer J5.3
- net MIC_WS: no longer MK1.1 (WS), R3.2
- new net: MK1.1 (WS), R3.2
- no-connect marks 5 -> 1
Other:
- moved on the sheet: C2, C3, C5, C6, C7, C8, FB1, FB2, J4, MK1, R1, R2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
