File: hardware/rev-b/intercom.kicad_sch (KiCad schematic)
At the start: 17 parts, among them J1 Conn_01x02, J4 PTT BREAKOUT, J5 VOLUME BREAKOUT, U1 MAX98357AETE+T

Commit message: Fix rev-B JLCPCB LCSC codes so they match the footprints.
Co-authored-by: Cursor <cursoragent@cursor.com>
Parts:
- C2: LCSC C28323 -> C29266; MPN CL21B105KBFNNNE -> CL05A105KO5NNNC; Manufacturer Samsung Electro-Mechanics -> Samsung
- C3, C5, C6: LCSC C107145 -> C3887425; MPN CC0805KRX7R9BB221 -> CL03B221KA3NNNC; Manufacturer YAGEO -> Samsung
- C7: LCSC C49678 -> C307382; MPN CC0805KRX7R9BB104 -> CL03A104KP3NN5C; Manufacturer YAGEO -> Samsung
- C8: LCSC C15850 -> C92487; MPN CL21A106KAYNNNE -> CL10A106MO8NQNC; Manufacturer Samsung Electro-Mechanics -> Samsung
- D1: LCSC (none) -> C1322304; MPN (none) -> HS-0402-UR; Manufacturer (none) -> Hongzhi Forest
- J1, J4: LCSC (none) -> C295747; MPN (none) -> S2B-PH-SM4-TB(LF)(SN); Manufacturer (none) -> JST
- J5: LCSC (none) -> C20089272; MPN (none) -> S3B-PH-SM4-TB; Manufacturer (none) -> JST
- MK1: LCSC (none) -> C5656610; MPN (none) -> ICS-43434; Manufacturer (none) -> TDK InvenSense
- R1: LCSC C17513 -> C270365; MPN 0805W8F1001T5E -> 0201WMF1001TEE
- R2: LCSC C17414 -> C473048; MPN 0805W8F1002T5E -> 0201WMF1002TEE
- R3: LCSC C17802 -> C473537; MPN 0805W8F680JT5E -> 0201WMF680JTEE
- U1: LCSC (none) -> C910544; MPN (none) -> MAX98357AETE+T; Manufacturer (none) -> Analog Devices
