File: hardware/rev-b/mcu.kicad_sch (KiCad schematic)
At the start: 15 parts, among them J2 USB_C_Receptacle_USB2.0_16P, J3 UART TEST PADS, SW3 KMR231GLFS, SW4 KMR231GLFS, U3 ESP32-S3-WROOM-1-N8R8, U6 USBLC6-2SC6

Commit message: Fix rev-B JLCPCB LCSC codes so they match the footprints.
Co-authored-by: Cursor <cursoragent@cursor.com>
Parts:
- C40, C47: LCSC (none) -> C92487; MPN (none) -> CL10A106MO8NQNC; Manufacturer (none) -> Samsung
- C41, C48: LCSC (none) -> C307382; MPN (none) -> CL03A104KP3NN5C; Manufacturer (none) -> Samsung
- C42: LCSC (none) -> C29266; MPN (none) -> CL05A105KO5NNNC; Manufacturer (none) -> Samsung
- J2: LCSC (none) -> C165948; MPN (none) -> TYPE-C-31-M-12; Manufacturer (none) -> HRO
- R40, R41: LCSC (none) -> C270344; MPN (none) -> 0201WMF5101TEE; Manufacturer (none) -> UNI-ROYAL
- R42, R43: LCSC (none) -> C473048; MPN (none) -> 0201WMF1002TEE; Manufacturer (none) -> UNI-ROYAL
- SW3, SW4: LCSC (none) -> C99271; MPN (none) -> KMR231GLFS; Manufacturer (none) -> C&K
- U3: LCSC (none) -> C2913201; MPN (none) -> ESP32-S3-WROOM-1-N8R8; Manufacturer (none) -> Espressif
- U6: LCSC (none) -> C7519; MPN (none) -> USBLC6-2SC6; Manufacturer (none) -> STMicroelectronics
