File: hardware/rev-b/power.kicad_sch (KiCad schematic)
At the start: 19 parts, among them SW2 JS102011SAQN, U2 TPS61088RHLR

Commit message: Fix rev-B JLCPCB LCSC codes so they match the footprints.
Co-authored-by: Cursor <cursoragent@cursor.com>
Parts:
- BT2: LCSC (none) -> C295747; MPN (none) -> S2B-PH-SM4-TB(LF)(SN); Manufacturer (none) -> JST
- C22, C31: LCSC C49678 -> C307382; MPN CC0805KRX7R9BB104 -> CL03A104KP3NN5C; Manufacturer YAGEO -> Samsung
- C23: LCSC C28323 -> C29266; MPN CL21B105KBFNNNE -> CL05A105KO5NNNC; Manufacturer Samsung Electro-Mechanics -> Samsung
- C24: LCSC C53134 -> C880416; MPN CL21B473KBCNNNC -> 0201X473K100NT; Manufacturer Samsung Electro-Mechanics -> Fenghua
- C25: LCSC C1744 -> C285054; MPN 0805B472K500NT -> 0201B472K100NT; Manufacturer FH -> Fenghua
- C26: LCSC C14857 -> C62546; MPN CL21C470JBANNNC -> 0201CG470J500NT; Manufacturer Samsung Electro-Mechanics -> Fenghua
- C27, C28, C29: LCSC C12891 -> C45783; MPN CL31A226KAHNNNE -> CL21A226MAQNNNE; Manufacturer Samsung Electro-Mechanics -> Samsung
- C30: LCSC C15850 -> C92487; MPN CL21A106KAYNNNE -> CL10A106MO8NQNC; Manufacturer Samsung Electro-Mechanics -> Samsung
- L2: LCSC (none) -> C7471471; MPN (none) -> XAL5030-122MEC; Manufacturer (none) -> Coilcraft
- R20, R21: LCSC C17539 -> C62188; MPN 0805W8F2003T5E -> 0201WMF2003TCE
- R22: LCSC C17501 -> C473559; MPN 0805W8F1803T5E -> 0201WMF1803TEE
- R23: LCSC C17756 -> C473524; MPN 0805W8F5602T5E -> 0201WMF5602TEE
- R24: LCSC C17414 -> C473048; MPN 0805W8F1002T5E -> 0201WMF1002TEE
- SW2: LCSC (none) -> C221660; MPN (none) -> JS102011SAQN; Manufacturer (none) -> C&K
- U2: LCSC (none) -> C87357; MPN (none) -> TPS61088RHLR; Manufacturer (none) -> Texas Instruments
Changed lines of the file:
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@@
 			)
 		)
-		(property "LCSC" "C49678"
+		(property "LCSC" "C307382"
 			(at 133.35 106.68 0)
 			(hide yes)
@@
 			)
 		)
-		(property "MPN" "CC0805KRX7R9BB104"
+		(property "MPN" "CL03A104KP3NN5C"
 			(at 133.35 106.68 0)
 			(hide yes)
@@
 			)
 		)
-		(property "Manufacturer" "YAGEO"
+		(property "Manufacturer" "Samsung"
 			(at 133.35 106.68 0)
 			(hide yes)
@@
 			)
 		)
-		(property "LCSC" "C14857"
+		(property "LCSC" "C62546"
 			(at 175.26 119.38 0)
 			(hide yes)
@@
 			)
 		)
-		(property "MPN" "CL21C470JBANNNC"
+		(property "MPN" "0201CG470J500NT"
 			(at 175.26 119.38 0)
 			(hide yes)
@@
 			)
 		)
-		(property "Manufacturer" "Samsung Electro-Mechanics"
+		(property "Manufacturer" "Fenghua"
 			(at 175.26 119.38 0)
 			(hide yes)
@@
 			)
 		)
-		(property "LCSC" "C12891"
+		(property "LCSC" "C45783"
 			(at 208.28 100.33 0)
 			(hide yes)
@@
 			)
 		)
-		(property "MPN" "CL31A226KAHNNNE"
+		(property "MPN" "CL21A226MAQNNNE"
 			(at 208.28 100.33 0)
 			(hide yes)
@@
 			)
 		)
-		(property "Manufacturer" "Samsung Electro-Mechanics"
+		(property "Manufacturer" "Samsung"
 			(at 208.28 100.33 0)
 			(hide yes)
@@
 			)
 		)
+		(property "Manufacturer" "Texas Instruments"
+			(at 154.94 91.44 0)
+			(hide yes)
+			(show_name no)
+			(do_not_autoplace no)
+			(effects
+				(font
+					(size 1.27 1.27)
+				)
+			)
+		)
+		(property "MPN" "TPS61088RHLR"
+			(at 154.94 91.44 0)
+			(hide yes)
+			(show_name no)
+			(do_not_autoplace no)
+			(effects
+				(font
+					(size 1.27 1.27)
+				)
+			)
+		)
+		(property "LCSC" "C87357"
+			(at 154.94 91.44 0)
+			(hide yes)
+			(show_name no)
+			(do_not_autoplace no)
+			(effects
+				(font
+					(size 1.27 1.27)
+				)
+			)
+		)
 		(pin "1"
 		)
@@
 			)
 		)
-		(property "LCSC" "C15850"
+		(property "LCSC" "C92487"
 			(at 101.6 99.06 0)
 			(hide yes)
@@
 			)
 		)
-		(property "MPN" "CL21A106KAYNNNE"
+		(property "MPN" "CL10A106MO8NQNC"
 			(at 101.6 99.06 0)
 			(hide yes)
@@
 			)
 		)
-		(property "Manufacturer" "Samsung Electro-Mechanics"
+		(property "Manufacturer" "Samsung"
 			(at 101.6 99.06 0)
 			(hide yes)
@@
 			)
 		)
-		(property "LCSC" "C53134"
+		(property "LCSC" "C880416"
 			(at 200.66 100.33 0)
 			(hide yes)
@@
 			)
 		)
-		(property "MPN" "CL21B473KBCNNNC"
+		(property "MPN" "0201X473K100NT"
 			(at 200.66 100.33 0)
 			(hide yes)
@@
 			)
 		)
-		(property "Manufacturer" "Samsung Electro-Mechanics"
+		(property "Manufacturer" "Fenghua"
 			(at 200.66 100.33 0)
 			(hide yes)
@@
 			)
 		)
-		(property "Datasheet" "https://www.ckswitches.com/media/1428/os.pdf"
+		(property "Datasheet" "https://www.ckswitches.com/media/1423/js.pdf"
+			(at 87.63 86.36 0)
+			(hide yes)
+			(show_name no)
+			(do_not_autoplace no)
+			(effects
+				(font
+					(size 1.27 1.27)
+				)
+			)
+		)
+		(property "Description" "C&K JS102011SAQN SMT right-angle SPDT slide. LCSC C221660."
+			(at 87.63 86.36 0)
+			(hide yes)
+			(show_name no)
+			(do_not_autoplace no)
+			(effects
+				(font
+					(size 1.27 1.27)
+				)
+			)
+		)
+		(property "Manufacturer" "C&K"
+			(at 87.63 86.36 0)
+			(hide yes)
+			(show_name no)
+			(do_not_autoplace no)
+			(effects
+				(font
+					(size 1.27 1.27)
+				)
+			)
+		)
+		(property "MPN" "JS102011SAQN"
 			(at 87.63 86.36 0)
 			(hide yes)
@@
 			)
 		)
-		(property "Description" "C&K OS102011MA1Q right-angle SPDT slide (side-facing). Order OS102011MA1QN1."
+		(property "LCSC" "C221660"
 			(at 87.63 86.36 0)
 			(hide yes)
@@
 			)
 		)
-		(property "LCSC" "C1744"
+		(property "LCSC" "C285054"
 			(at 196.85 119.38 0)
 			(hide yes)
@@
 			)
 		)
-		(property "MPN" "0805B472K500NT"
+		(property "MPN" "0201B472K100NT"
 			(at 196.85 119.38 0)
 			(hide yes)
@@
 			)
 		)
-		(property "Manufacturer" "FH"
+		(property "Manufacturer" "Fenghua"
 			(at 196.85 119.38 0)
 			(hide yes)
@@
 			)
 		)
-		(property "LCSC" "C17414"
+		(property "LCSC" "C473048"
 			(at 182.88 88.9 0)
 			(hide yes)
@@
 			)
 		)
-		(property "MPN" "0805W8F1002T5E"
+		(property "MPN" "0201WMF1002TEE"
 			(at 182.88 88.9 0)
 			(hide yes)
@@
 			)
 		)
-		(property "LCSC" "C17501"
+		(property "LCSC" "C473559"
 			(at 214.63 86.36 0)
 			(hide yes)
@@
 			)
 		)
-		(property "MPN" "0805W8F1803T5E"
+		(property "MPN" "0201WMF1803TEE"
 			(at 214.63 86.36 0)
 			(hide yes)
@@
 			)
 		)
-		(property "LCSC" "C49678"
+		(property "LCSC" "C307382"
 			(at 111.76 99.06 0)
 			(hide yes)
@@
 			)
 		)
-		(property "MPN" "CC0805KRX7R9BB104"
+		(property "MPN" "CL03A104KP3NN5C"
 			(at 111.76 99.06 0)
 			(hide yes)
@@
 			)
 		)
-		(property "Manufacturer" "YAGEO"
+		(property "Manufacturer" "Samsung"
 			(at 111.76 99.06 0)
 			(hide yes)
@@
 			)
 		)
-		(property "LCSC" "C12891"
+		(property "LCSC" "C45783"
 			(at 187.96 109.22 0)
 			(hide yes)
@@
 			)
 		)
-		(property "MPN" "CL31A226KAHNNNE"
+		(property "MPN" "CL21A226MAQNNNE"
 			(at 187.96 109.22 0)
 			(hide yes)
@@
 			)
 		)
-		(property "Manufacturer" "Samsung Electro-Mechanics"
+		(property "Manufacturer" "Samsung"
 			(at 187.96 109.22 0)
 			(hide yes)
@@
 			)
 		)
-		(property "LCSC" "C17539"
+		(property "LCSC" "C62188"
 			(at 133.35 96.52 0)
 			(hide yes)
@@
 			)
 		)
-		(property "MPN" "0805W8F2003T5E"
+		(property "MPN" "0201WMF2003TCE"
 			(at 133.35 96.52 0)
 			(hide yes)
@@
 			)
 		)
-		(property "LCSC" "C17756"
+		(property "LCSC" "C473524"
 			(at 214.63 76.2 0)
 			(hide yes)
@@
 			)
 		)
-		(property "MPN" "0805W8F5602T5E"
+		(property "MPN" "0201WMF5602TEE"
 			(at 214.63 76.2 0)
 			(hide yes)
@@
 			)
 		)
+		(property "Manufacturer" "JST"
+			(at 73.66 86.36 0)
+			(hide yes)
+			(show_name no)
+			(do_not_autoplace no)
+			(effects
+				(font
+					(size 1.27 1.27)
+				)
+			)
+		)
+		(property "MPN" "S2B-PH-SM4-TB(LF)(SN)"
+			(at 73.66 86.36 0)
+			(hide yes)
+			(show_name no)
+			(do_not_autoplace no)
+			(effects
+				(font
+					(size 1.27 1.27)
+				)
+			)
+		)
+		(property "LCSC" "C295747"
+			(at 73.66 86.36 0)
+			(hide yes)
+			(show_name no)
+			(do_not_autoplace no)
+			(effects
+				(font
+					(size 1.27 1.27)
+				)
+			)
+		)
 		(pin "1"
 		)
@@
 			)
 		)
-		(property "LCSC" "C28323"
+		(property "LCSC" "C29266"
 			(at 179.07 109.22 0)
 			(hide yes)
@@
 			)
 		)
-		(property "MPN" "CL21B105KBFNNNE"
+		(property "MPN" "CL05A105KO5NNNC"
 			(at 179.07 109.22 0)
 			(hide yes)
@@
 			)
 		)
-		(property "Manufacturer" "Samsung Electro-Mechanics"
+		(property "Manufacturer" "Samsung"
 			(at 179.07 109.22 0)
 			(hide yes)
@@
 			)
 		)
+		(property "Manufacturer" "Coilcraft"
+			(at 124.46 91.44 0)
+			(hide yes)
+			(show_name no)
+			(do_not_autoplace no)
+			(effects
+				(font
+					(size 1.27 1.27)
+				)
+			)
+		)
+		(property "MPN" "XAL5030-122MEC"
+			(at 124.46 91.44 0)
+			(hide yes)
+			(show_name no)
+			(do_not_autoplace no)
+			(effects
+				(font
+					(size 1.27 1.27)
+				)
+			)
+		)
+		(property "LCSC" "C7471471"
+			(at 124.46 91.44 0)
+			(hide yes)
+			(show_name no)
+			(do_not_autoplace no)
+			(effects
+				(font
+					(size 1.27 1.27)
+				)
+			)
+		)
 		(pin "1"
 		)
@@
 			)
 		)
-		(property "LCSC" "C12891"
+		(property "LCSC" "C45783"
 			(at 204.47 119.38 0)
 			(hide yes)
@@
 			)
 		)
-		(property "MPN" "CL31A226KAHNNNE"
+		(property "MPN" "CL21A226MAQNNNE"
 			(at 204.47 119.38 0)
 			(hide yes)
@@
 			)
 		)
-		(property "Manufacturer" "Samsung Electro-Mechanics"
+		(property "Manufacturer" "Samsung"
 			(at 204.47 119.38 0)
 			(hide yes)
@@
 			)
 		)
-		(property "LCSC" "C17539"
+		(property "LCSC" "C62188"
 			(at 233.68 91.44 0)
 			(hide yes)
@@
 			)
 		)
-		(property "MPN" "0805W8F2003T5E"
+		(property "MPN" "0201WMF2003TCE"
 			(at 233.68 91.44 0)
 			(hide yes)
