File: hardware/rev-b/usb_power.kicad_sch (KiCad schematic)
At the start: 11 parts, among them U4 AP2112K-3.3TRG1, U5 MCP73831T-2ACI/OT

Commit message: Fix rev-B JLCPCB LCSC codes so they match the footprints.
Co-authored-by: Cursor <cursoragent@cursor.com>
Parts:
- C43, C44: LCSC (none) -> C29266; MPN (none) -> CL05A105KO5NNNC; Manufacturer (none) -> Samsung
- C45, C46: LCSC (none) -> C23733; MPN (none) -> CL05A475MP5NRNC; Manufacturer (none) -> Samsung
- C49: LCSC (none) -> C92487; MPN (none) -> CL10A106MO8NQNC; Manufacturer (none) -> Samsung
- D2: LCSC (none) -> C727060; MPN (none) -> SS34; Manufacturer (none) -> TWGMC
- D3: LCSC (none) -> C1322308; MPN (none) -> HS-0402-UG; Manufacturer (none) -> Hongzhi Forest
- R44: LCSC (none) -> C270358; MPN (none) -> 0201WMF2001TEE; Manufacturer (none) -> UNI-ROYAL
- R45: LCSC (none) -> C270365; MPN (none) -> 0201WMF1001TEE; Manufacturer (none) -> UNI-ROYAL
- U4: LCSC (none) -> C51118; MPN (none) -> AP2112K-3.3TRG1; Manufacturer (none) -> Diodes Incorporated
- U5: LCSC (none) -> C424093; MPN (none) -> MCP73831T-2ACI/OT; Manufacturer (none) -> Microchip
